File: schematics/EVA1_production/TRAM.kicad_sch (KiCad schematic)
At the start: 13 parts, among them U1 HY6264AxP, U10 74LS166, U2 74LS573, U3 27C32, U31 74LS32, U5 74LS245, U6 74LS157, U7 74LS157, U8 74LS157, U9 27C64

Commit message: New version for production
Other:
- note added: "check why there is a strange rollover when A11 is connected!"
- note added: "when grounding A11 everything is fine!"
Changed lines of the file:
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@@
+		)
+	)
+	(text "when grounding A11 everything is fine!"
+		(exclude_from_sim no)
+		(at 125.476 51.562 0)
+		(effects
+			(font
+				(size 1.27 1.27)
+			)
 		)
 	)
@@
 		(effects
 			(font
+				(size 1.27 1.27)
+			)
+		)
+	)
+	(text "check why there is a strange \nrollover when A11 is connected!"
+		(exclude_from_sim no)
+		(at 13.97 140.97 0)
+		(effects
+			(font
