File: schematics/EVA1_production/videosignal.kicad_sch (KiCad schematic)
At the start: 21 parts, among them J2 BAS, Q2 BC337, Q3 BC337, U12 74LS32, U18 74LS08, U19 74LS86, U22 74LS04, U37 74LS08, U4 74LS74

Commit message: New version for production
Parts:
- R3: value 47E -> 560E
- R9: value 560E -> 47E
Other:
- note removed: "ch. R9 to 560E and R3 to 47E!"
Changed lines of the file:
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@@
-		)
-	)
-	(text "ch. R9 to 560E\nand R3 to 47E!"
-		(exclude_from_sim no)
-		(at 278.892 175.006 0)
-		(effects
-			(font
-				(size 1.27 1.27)
-			)
-			(justify left)
 		)
 	)
@@
 			)
 		)
-		(property "Value" "47E"
+		(property "Value" "560E"
 			(at 151.13 137.16 90)
 			(effects
@@
 			)
 		)
-		(property "Value" "560E"
+		(property "Value" "47E"
 			(at 165.1 111.76 90)
 			(effects
