File: schematics/EVA1_v2/EVA1_v2.kicad_pcb (KiCad board)
At the start: 2 copper layers, 218 x 125 mm, 151 parts, among them J1 17, J10 Micro_SD_Card_Det2, J11 Conn_01x02, J2 BAS, J3 DE15_Plug_HighDensity_Mountin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, J4 HX20, J5 TF20, J6 9, J7 8, J8 Barrel_Jack_Switch, J9 Converter, Q2 BC337, Q3 BC337, SW1 PX_CLK_BTN, SW2 AUTO_ADJUST, U1 HY6264AxP, U10 74LS165, U11 CY62256-70PC, U12 74LS32, U13 74LS221, U14 74LS573, U15 MC6803, U16 MC6845, U17 27C256, U18 74LS08, U19 74LS86, U2 74LS573, U20 74LS290, U21 Sparkfun_Pro_Micro, U22 74F14, U23 74LS74, U24 74LS74, U25 74LS157, U26 74LS157, U27 74LS157, U28 74LS157, U29 74LS107, U3 27C32, U30 MAX232, U31 74LVC08, U32 GAL16V8, U33 AMS1117-3.3, U34 RaspberryPi_Pico, U35 74LS165, U36 74LS245, U37 74LVC08, U38 74LS573, U4 74LS74, U45 GAL16V8, U5 74LS245, U6 74LS157, U7 74LS157, U8 74LS157, U9 27C64, Y2 19M66, Y3 19M66

Commit message: schematics updated
Parts:
- removed R102: 4k7, Resistor_SMD:R_1206_3216Metric_Pad1.30x1.75mm_HandSolder
- removed R2: 4k7, Resistor_THT:R_Axial_DIN0411_L9.9mm_D3.6mm_P12.70mm_Horizontal
- added JP10: SolderJumper_2_Open, Jumper:SolderJumper-2_P1.3mm_Open_RoundedPad1.0x1.5mm, F.Cu at (145.4, 108.6)
- added JP9: SCLK*2, Connector_PinHeader_2.54mm:PinHeader_1x03_P2.54mm_Vertical, F.Cu at (224.3, 128.9)
- JP7: value SolderJumper_3_Bridged12 -> TA11_on_off
- turned JP5 to 0 degrees
Connections:
- JP5 pad 1: /VS -> GND
- JP5 pad 3: GND -> /VS
- R1 pad 1: GND -> +5V
- R5 pad 1: GND -> +5V
- U17 pad 1: unconnected-(U17-VPP-Pad1) -> Net-(JP10-B)
- U17 pad 26: Net-(U17-A13) -> /A13
- U2 pad 1: +5V -> GND
- U20 pad 11: Net-(U20-Cp1) -> Net-(JP9-C)
- U20 pad 9: Net-(U20-Cp1) -> Net-(JP9-B)
- U38 pad 1: +5V -> GND
- U38 pad 11: /Graphic RAM, MUX and Shiftregister/LTDAT -> /LTDAT
Routing:
- net /LTDAT: track 219.6 -> 252.8 mm
- net Net-(JP9-B): track 0.00 -> 31.9 mm, vias 0 -> 1
- net Net-(JP9-C): track 0.00 -> 24.9 mm, vias 0 -> 1
- net GND: track 1816.6 -> 1838.3 mm
- net /A13: track 161.2 -> 174.5 mm, vias 3 -> 4
- net Net-(U17-A13): track 11.2 -> 0.00 mm
- net +5V: track 1426.7 -> 1434.5 mm, vias 29 -> 28
- net Net-(U20-Cp1): track 7.41 -> 0.00 mm
- net /RASCLKIN: track 19.5 -> 26.0 mm
- net Net-(JP10-B): track 0.00 -> 3.35 mm
- net /A2: track 239.5 -> 237.3 mm
- net /GDAT: track 56.5 -> 58.3 mm
- net /Din: track 152.9 -> 151.3 mm
- net /E: track 232.1 -> 231.0 mm
- net /V4: track 138.8 -> 137.8 mm
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Other:
- board text added: "38.4 BAUD 76.8"

Commit message: New version for production
Parts:
- added H8: M3, MountingHole:MountingHole_3.2mm_M3, F.Cu at (29.0, 30.8)
- added H9: M3, MountingHole:MountingHole_3.2mm_M3, F.Cu at (29.0, 130.2)
- C5: moved to B.Cu
- J11: value Conn_01x02 -> Conn_Coaxial; footprint Connector_PinHeader_2.54mm:PinHeader_1x02_P2.54mm_Vertical -> my_own_conn:Keystone_RCA-Jack
- SW1, SW2: footprint Button_Switch_THT:SW_PUSH_6mm -> Button_Switch_THT:SW_Tactile_SPST_Angled_PTS645Vx83-2LFS
- moved H6 119.0 mm to (229.0, 130.2)
- moved H2 119.0 mm to (229.0, 30.8)
- moved SW1 51.8 mm to (86.1, 141.1), turned to 180 degrees
- moved U37 50.6 mm to (31.1, 116.9), turned to 90 degrees
- moved C5 39.9 mm to (122.7, 101.1), turned to 0 degrees
- moved C108 27.7 mm to (126.7, 126.5)
- moved C8 27.7 mm to (126.7, 124.0)
- moved U33 22.6 mm to (119.9, 127.3)
- moved J9 16.4 mm to (88.4, 126.5)
- moved J11 13.2 mm to (141.0, 142.0)
- moved SW2 6.31 mm to (41.0, 141.1), turned to 180 degrees
- moved C17 5.56 mm to (218.2, 25.4)
- moved JP9 5.41 mm to (218.9, 129.8)
- moved H5 3.58 mm to (226.5, 130.2)
- moved H3 3.51 mm to (226.5, 30.8)
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Connections:
- J11 pad 1: +5V -> Net-(J11-In)
- J2 pad 1: Net-(J2-Pin_1) -> Net-(J11-In)
- Q2 pad 3: Net-(J2-Pin_1) -> Net-(J11-In)
- R8 pad 1: Net-(J2-Pin_1) -> Net-(J11-In)
- U37 pad 1: /Video -> /HS
- U37 pad 11: Net-(U34-GP7) -> /SB
- U37 pad 12: /HS -> /Video
- U37 pad 13: /HS -> /Video
- U37 pad 2: /Video -> /HS
- U37 pad 3: /SB -> Net-(U34-GP7)
Routing:
- net Net-(J11-In): track 0.00 -> 58.0 mm
- net Net-(J2-Pin_1): track 49.0 -> 0.00 mm
- net +5V: track 1434.5 -> 1387.8 mm, vias 28 -> 27
- net Net-(U34-GP7): track 58.1 -> 15.3 mm
- net /INTENS: track 84.6 -> 126.5 mm
- net /TX: track 164.9 -> 123.7 mm, vias 5 -> 3
- net /SB: track 79.9 -> 41.0 mm
- net /VS#: track 50.7 -> 86.5 mm, vias 2 -> 1
- net Net-(U34-GP22): track 35.1 -> 67.6 mm, vias 0 -> 1
- net /HS: track 85.2 -> 114.9 mm, vias 1 -> 0
- net Net-(U34-GP6): track 46.7 -> 17.6 mm
- net /Video: track 149.6 -> 176.8 mm, vias 4 -> 3
- net /SG_INT: track 83.9 -> 67.6 mm
- net Net-(U30-VS+): track 19.9 -> 34.0 mm
- net +3V3: track 208.3 -> 195.0 mm, vias 4 -> 6
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Other:
- board text added: "BAS"
- board text added: "Gehäuse"
- board text removed: "PWR BAS"
