File: schematics/EVA1_v2/EVA1_v2.kicad_pcb (KiCad board)
At the start: 2 copper layers, 218 x 125 mm, 153 parts, among them J1 17, J10 Micro_SD_Card_Det2, J11 Conn_Coaxial, J2 BAS, J3 DE15_Plug_HighDensity_Mountin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, J4 HX20, J5 TF20, J6 9, J7 8, J8 Barrel_Jack_Switch, J9 Converter, Q2 BC337, Q3 BC337, SW1 PX_CLK_BTN, SW2 AUTO_ADJUST, U1 HY6264AxP, U10 74LS165, U11 CY62256-70PC, U12 74LS32, U13 74LS221, U14 74LS573, U15 MC6803, U16 MC6845, U17 27C256, U18 74LS08, U19 74LS86, U2 74LS573, U20 74LS290, U21 Sparkfun_Pro_Micro, U22 74F14, U23 74LS74, U24 74LS74, U25 74LS157, U26 74LS157, U27 74LS157, U28 74LS157, U29 74LS107, U3 27C32, U30 MAX232, U31 74LVC08, U32 GAL16V8, U33 AMS1117-3.3, U34 RaspberryPi_Pico, U35 74LS165, U36 74LS245, U37 74LVC08, U38 74LS573, U4 74LS74, U45 GAL16V8, U5 74LS245, U6 74LS157, U7 74LS157, U8 74LS157, U9 27C64, Y2 19M66, Y3 19M66

Commit message: Schematic and Board updated
Parts:
- added J12: Conn_01x06, Connector_PinSocket_2.54mm:PinSocket_1x06_P2.54mm_Vertical, F.Cu at (50.0, 129.9)
- added J13: Conn_01x02, Connector_PinSocket_2.54mm:PinSocket_1x02_P2.54mm_Vertical, F.Cu at (43.7, 129.9)
- added R2: 10k, Resistor_SMD:R_1206_3216Metric_Pad1.30x1.75mm_HandSolder, F.Cu at (46.9, 104.8)
- added R25: 10k, Resistor_SMD:R_1206_3216Metric_Pad1.30x1.75mm_HandSolder, F.Cu at (24.7, 121.2)
- added R26: 10k, Resistor_SMD:R_1206_3216Metric_Pad1.30x1.75mm_HandSolder, F.Cu at (60.3, 121.0)
- added R27: 10k, Resistor_SMD:R_1206_3216Metric_Pad1.30x1.75mm_HandSolder, F.Cu at (57.9, 121.0)
- added R28: 10k, Resistor_SMD:R_1206_3216Metric_Pad1.30x1.75mm_HandSolder, F.Cu at (34.7, 121.2)
- added R29: 10k, Resistor_SMD:R_1206_3216Metric_Pad1.30x1.75mm_HandSolder, F.Cu at (62.7, 121.0)
- U10, U35: value 74LS165 -> 74HCT165
- U12: value 74LS32 -> 74HCT32
- U18: value 74LS08 -> 74HCT08
- U19: value 74LS86 -> 74HCT86
- U22: value 74F14 -> 74HCT14
- U23, U24, U4: value 74LS74 -> 74HCT74
- U25, U26, U27, U28, U6, U7, U8: value 74LS157 -> 74ALS157
- U36, U5: value 74LS245 -> 74HCT245
- Y2, Y3: value 19M66 -> 18M432
Connections:
- U34 pad 12: unconnected-(U34-GP9-Pad12) -> /PB
- U34 pad 15: unconnected-(U34-GP11-Pad15) -> /PG
- U34 pad 17: unconnected-(U34-GP13-Pad17) -> /PR
- U34 pad 2: unconnected-(U34-GP1-Pad2) -> /PB
- U34 pad 5: unconnected-(U34-GP3-Pad5) -> /PG
- U34 pad 6: unconnected-(U34-GP4-Pad6) -> /SR
- U34 pad 7: unconnected-(U34-GP5-Pad7) -> /PR
- U37 pad 11: /SB -> /VID
- U37 pad 8: /SG_INT -> /INT
Routing:
- net /PB: track 0.00 -> 45.7 mm
- net /PG: track 0.00 -> 43.8 mm, vias 0 -> 1
- net /PR: track 0.00 -> 39.4 mm, vias 0 -> 1
- net /INT: track 0.00 -> 36.6 mm, vias 0 -> 1
- net /SR: track 0.00 -> 35.7 mm, vias 0 -> 1
- net /VID: track 0.00 -> 30.7 mm, vias 0 -> 2
- net GND: track 1831.8 -> 1858.7 mm
- net /SB: track 41.0 -> 62.8 mm
- net /SG_INT: track 67.6 -> 61.7 mm
- net Net-(U34-GP22): track 67.6 -> 64.6 mm, vias 1 -> 2
- net +3V3: track 195.0 -> 192.1 mm
Other:
- board text added: "EVA1 v2 v0.5"
- board text added: "SB PB SG PG SR PR"
- board text added: "VID INT"

Commit message: new Gerber files
Parts:
- removed U38: 74LS573, Package_DIP:DIP-20_W7.62mm
- renumbered C20 to C114
Connections:
- U35 pad 11: /Graphic RAM, MUX and Shiftregister/LD0 -> /Graphic RAM, MUX and Shiftregister/GD0
- U35 pad 12: /Graphic RAM, MUX and Shiftregister/LD1 -> /Graphic RAM, MUX and Shiftregister/GD1
- U35 pad 13: /Graphic RAM, MUX and Shiftregister/LD2 -> /Graphic RAM, MUX and Shiftregister/GD2
- U35 pad 14: /Graphic RAM, MUX and Shiftregister/LD3 -> /Graphic RAM, MUX and Shiftregister/GD3
- U35 pad 3: /Graphic RAM, MUX and Shiftregister/LD4 -> /Graphic RAM, MUX and Shiftregister/GD4
- U35 pad 4: /Graphic RAM, MUX and Shiftregister/LD5 -> /Graphic RAM, MUX and Shiftregister/GD5
- U35 pad 5: /Graphic RAM, MUX and Shiftregister/LD6 -> /Graphic RAM, MUX and Shiftregister/GD6
- U35 pad 6: /Graphic RAM, MUX and Shiftregister/LD7 -> /Graphic RAM, MUX and Shiftregister/GD7
Routing:
- net /LTDAT: track 252.8 -> 219.6 mm
- net GND: track 1858.7 -> 1834.1 mm
- net /Graphic RAM, MUX and Shiftregister/LD7: track 24.1 -> 0.00 mm, vias 1 -> 0
- net /Graphic RAM, MUX and Shiftregister/GD7: track 38.0 -> 61.7 mm, vias 1 -> 3
- net /Graphic RAM, MUX and Shiftregister/GD6: track 33.6 -> 55.5 mm, vias 1 -> 3
- net /Graphic RAM, MUX and Shiftregister/GD2: track 46.6 -> 66.8 mm
- net /Graphic RAM, MUX and Shiftregister/GD3: track 42.2 -> 62.2 mm
- net /Graphic RAM, MUX and Shiftregister/GD1: track 39.3 -> 58.8 mm
- net /Graphic RAM, MUX and Shiftregister/GD0: track 37.3 -> 56.5 mm
- net /Graphic RAM, MUX and Shiftregister/LD6: track 17.8 -> 0.00 mm, vias 1 -> 0
- net /Graphic RAM, MUX and Shiftregister/GD5: track 33.0 -> 50.3 mm
- net /Graphic RAM, MUX and Shiftregister/LD2: track 12.4 -> 0.00 mm
- net /Graphic RAM, MUX and Shiftregister/LD3: track 12.4 -> 0.00 mm
- net /Graphic RAM, MUX and Shiftregister/LD1: track 12.3 -> 0.00 mm
- net /Graphic RAM, MUX and Shiftregister/LD0: track 12.3 -> 0.00 mm
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