File: schematics/EVA1_v2/EVA1_v2.kicad_sch (KiCad schematic)
At the start: 75 parts, among them J1 17, J10 Micro_SD_Card_Det2, J3 DE15_Plug_HighDensity_Mountin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, J4 HX20, J5 TF20, J6 9, J7 8, J9 Converter, SW1 PX_CLK_BTN, SW2 AUTO_ADJUST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

Commit message: schematics updated
Parts:
- removed R102: 4k7, Resistor_SMD:R_1206_3216Metric_Pad1.30x1.75mm_HandSolder, symbol Device:R_Small
- removed R2: 4k7, Resistor_THT:R_Axial_DIN0411_L9.9mm_D3.6mm_P12.70mm_Horizontal, symbol Device:R_Small
- added JP10: SolderJumper_2_Open, Jumper:SolderJumper-2_P1.3mm_Open_RoundedPad1.0x1.5mm, symbol Jumper:SolderJumper_2_Open
- added JP9: SCLK*2, Connector_PinHeader_2.54mm:PinHeader_1x03_P2.54mm_Vertical, symbol Jumper:Jumper_3_Open
Connections:
- net +5V: now also R1.1, R5.1
- net A13: now also U17.26 (A13)
- net GND: now also JP5.1 (A), JP10.1 (A); no longer JP5.3 (B), R1.1, R5.1
- net RASCLKIN: now also JP9.1 (A)
- net VS: now also JP5.3 (B); no longer JP5.1 (A)
- net at U20.11 (Cp1): now also JP9.2 (C); no longer U20.9 (Q0)
- net at U17.1 (VPP): now also JP10.2 (B)
- new net: JP9.3 (B), U20.9 (Q0)
- no-connect marks 22 -> 21
Other:
- sheet Graphic RAM, MUX and Shiftregister ports: added LTDAT; removed none
- note added: "0xE000"
- note removed: "0xC000"
- moved on the sheet: R1, R5

Commit message: New version for production
Parts:
- added H8, H9: M3, MountingHole:MountingHole_3.2mm_M3, symbol Mechanical:MountingHole
- SW1, SW2: footprint Button_Switch_THT:SW_PUSH_6mm -> Button_Switch_THT:SW_Tactile_SPST_Angled_PTS645Vx83-2LFS
Connections:
- net HS: now also U37.1, U37.2; no longer U37.12, U37.13
- net SB: now also U37.11; no longer U37.3
- net Video: now also U37.12, U37.13; no longer U37.1, U37.2
- net at U34.10 (GP7): now also U37.3; no longer U37.11
Other:
- note added: "In: 3.08MHz"
- note removed: "In: 3.07MHz"
- moved on the sheet: H3, U37A, U37D

Commit message: Schematic and Board updated
Parts:
- added J12: Conn_01x06, Connector_PinSocket_2.54mm:PinSocket_1x06_P2.54mm_Vertical, symbol Connector_Generic:Conn_01x06
- added J13: Conn_01x02, Connector_PinSocket_2.54mm:PinSocket_1x02_P2.54mm_Vertical, symbol Connector_Generic:Conn_01x02
- added R2, R25, R26, R27, R28, R29: 10k, Resistor_SMD:R_1206_3216Metric_Pad1.30x1.75mm_HandSolder, symbol Device:R_Small
- U19: value 74LS86 -> 74HCT86
- U22: value 74F14 -> 74HCT14
- U23, U24: value 74LS74 -> 74HCT74
- Y2, Y3: value 19M66 -> 18M432
Connections:
- net GND: now also R2.2, R25.2, R26.2, R27.2, R28.2, R29.2
- net SB: now also J12.1 (Pin_1), R2.1; no longer U37.11
- net SG_INT: now also J12.3 (Pin_3), R26.1; no longer U37.8
- net PB: now reaches U34.12 (GP9)
- net PB: now also U34.2 (GP1), J12.2 (Pin_2), R25.1
- net PG: now reaches U34.15 (GP11)
- net PG: now also U34.5 (GP3), J12.4 (Pin_4), R27.1
- net PR: now reaches U34.17 (GP13)
- net PR: now also U34.7 (GP5), J12.6 (Pin_6), R29.1
- net SR: now reaches U34.6 (GP4)
- net SR: now also J12.5 (Pin_5), R28.1
- new net INT: J13.2 (Pin_2), U37.8
- new net VID: J13.1 (Pin_1), U37.11
Other:
- note added: "Problems and fixes for next Version: Arduino Pro micro doesn't work (crashes), '573 Latch on Graphics side is not necsessary, Color Input to Pi Pico is wrong,"
- moved on the sheet: U37C, U37D
