File: schematics/EVA1_v2/Power.kicad_sch (KiCad schematic)
At the start: 48 parts, among them J11 Conn_01x02, J8 Barrel_Jack_Switch, U12 74LS32, U13 74LS221, U18 74LS08, U19 74LS86, U22 74F14, U23 74LS74, U24 74LS74, U29 74LS107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

Commit message: New version for production
Parts:
- removed J11: Conn_01x02, Connector_PinHeader_2.54mm:PinHeader_1x02_P2.54mm_Vertical, symbol Connector_Generic:Conn_01x02
Changed lines of the file:
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@@
 (kicad_sch
-	(version 20231120)
+	(version 20250114)
 	(generator "eeschema")
-	(generator_version "8.0")
+	(generator_version "9.0")
 	(paper "A4")
 	(title_block
@@
 	(wire
 		(pts
-			(xy 81.28 36.83) (xy 83.82 36.83)
-		)
-		(stroke
-			(width 0)
-			(type default)
-		)
-	)
-	(wire
-		(pts
 			(xy 123.19 132.08) (xy 123.19 134.62)
 		)
@@
 	(wire
 		(pts
-			(xy 81.28 31.75) (xy 81.28 34.29)
-		)
-		(stroke
-			(width 0)
-			(type default)
-		)
-	)
-	(wire
-		(pts
 			(xy 191.77 100.33) (xy 194.31 100.33)
 		)
@@
 	(wire
 		(pts
-			(xy 81.28 38.1) (xy 81.28 36.83)
-		)
-		(stroke
-			(width 0)
-			(type default)
-		)
-	)
-	(wire
-		(pts
 			(xy 40.64 54.61) (xy 35.56 54.61)
 		)
@@
 	(wire
 		(pts
-			(xy 83.82 34.29) (xy 81.28 34.29)
-		)
-		(stroke
-			(width 0)
-			(type default)
-		)
-	)
-	(wire
-		(pts
 			(xy 27.94 116.84) (xy 36.83 116.84)
 		)
@@
 	)
 	(symbol
-		(lib_id "power:GND")
-		(at 81.28 38.1 0)
-		(unit 1)
-		(exclude_from_sim no)
-		(in_bom yes)
-		(on_board yes)
-		(dnp no)
-		(property "Reference" "#PWR160"
-			(at 81.28 44.45 0)
-			(effects
-				(font
-					(size 1.27 1.27)
-				)
-				(hide yes)
-			)
-		)
-		(property "Value" "GND"
-			(at 81.28 41.91 0)
-			(effects
-				(font
-					(size 1.27 1.27)
-				)
-			)
-		)
-		(property "Footprint" ""
-			(at 81.28 38.1 0)
-			(effects
-				(font
-					(size 1.27 1.27)
-				)
-				(hide yes)
-			)
-		)
-		(property "Datasheet" ""
-			(at 81.28 38.1 0)
-			(effects
-				(font
-					(size 1.27 1.27)
-				)
-				(hide yes)
-			)
-		)
-		(property "Description" ""
-			(at 81.28 38.1 0)
-			(effects
-				(font
-					(size 1.27 1.27)
-				)
-				(hide yes)
-			)
-		)
-		(pin "1"
-		)
-		(instances
-			(project "EVA1_v2"
-				(path "/5be3a086-9309-43f4-b37c-0519e88c3e26/8c3b0133-ca1d-4caf-84d5-fd69701054d3"
-					(reference "#PWR160")
-					(unit 1)
-				)
-			)
-		)
-	)
-	(symbol
 		(lib_id "power:+5V")
 		(at 111.76 132.08 0)
@@
 				)
 			)
-		)
-	)
-	(symbol
-		(lib_id "Connector_Generic:Conn_01x02")
-		(at 88.9 34.29 0)
-		(unit 1)
-		(exclude_from_sim no)
-		(in_bom yes)
-		(on_board yes)
-		(dnp no)
-		(fields_autoplaced yes)
-		(property "Reference" "J11"
-			(at 91.44 34.2899 0)
-			(effects
-				(font
-					(size 1.27 1.27)
-				)
-				(justify left)
-			)
-		)
-		(property "Value" "Conn_01x02"
-			(at 91.44 36.8299 0)
-			(effects
-				(font
-					(size 1.27 1.27)
-				)
-				(justify left)
-			)
-		)
-		(property "Footprint" "Connector_PinHeader_2.54mm:PinHeader_1x02_P2.54mm_Vertical"
-			(at 88.9 34.29 0)
-			(effects
-				(font
-					(size 1.27 1.27)
-				)
-				(hide yes)
-			)
-		)
-		(property "Datasheet" "~"
-			(at 88.9 34.29 0)
-			(effects
-				(font
-					(size 1.27 1.27)
-				)
-				(hide yes)
-			)
-		)
-		(property "Description" "Generic connector, single row, 01x02, script generated (kicad-library-utils/schlib/autogen/connector/)"
-			(at 88.9 34.29 0)
-			(effects
-				(font
-					(size 1.27 1.27)
-				)
-				(hide yes)
-			)
-		)
-		(pin "1"
-		)
-		(pin "2"
-		)
-		(instances
-			(project ""
-				(path "/5be3a086-9309-43f4-b37c-0519e88c3e26/8c3b0133-ca1d-4caf-84d5-fd69701054d3"
-					(reference "J11")
-					(unit 1)
-				)
-			)
-		)
-	)
-	(symbol
-		(lib_id "power:+5V")
-		(at 81.28 31.75 0)
-		(unit 1)
-		(exclude_from_sim no)
-		(in_bom yes)
-		(on_board yes)
-		(dnp no)
-		(property "Reference" "#PWR161"
-			(at 81.28 35.56 0)
-			(effects
-				(font
-					(size 1.27 1.27)
-				)
-				(hide yes)
-			)
-		)
-		(property "Value" "+5V"
-			(at 81.28 28.575 0)
-			(effects
-				(font
-					(size 1.27 1.27)
-				)
-			)
-		)
-		(property "Footprint" ""
-			(at 81.28 31.75 0)
-			(effects
-				(font
-					(size 1.27 1.27)
-				)
-				(hide yes)
-			)
-		)
-		(property "Datasheet" ""
-			(at 81.28 31.75 0)
-			(effects
-				(font
-					(size 1.27 1.27)
-				)
-				(hide yes)
-			)
-		)
-		(property "Description" ""
-			(at 81.28 31.75 0)
-			(effects
-				(font
-					(size 1.27 1.27)
-				)
-				(hide yes)
-			)
-		)
-		(pin "1"
-		)
-		(instances
-			(project "EVA1_v2"
-				(path "/5be3a086-9309-43f4-b37c-0519e88c3e26/8c3b0133-ca1d-4caf-84d5-fd69701054d3"
-					(reference "#PWR161")
-					(unit 1)
-				)
-			)

Commit message: Schematic and Board updated
Parts:
- U12: value 74LS32 -> 74HCT32
- U18: value 74LS08 -> 74HCT08
- U19: value 74LS86 -> 74HCT86
- U22: value 74F14 -> 74HCT14
- U23, U24, U4: value 74LS74 -> 74HCT74
Changed lines of the file:
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@@
 			)
 		)
-		(property "Value" "74LS32"
+		(property "Value" "74HCT32"
 			(at 234.95 114.3 0)
 			(effects
@@
 			)
 		)
-		(property "Value" "74F14"
+		(property "Value" "74HCT14"
 			(at 257.81 107.95 0)
 			(effects
@@
 			)
 		)
-		(property "Value" "74LS86"
+		(property "Value" "74HCT86"
 			(at 85.344 146.05 0)
 			(effects
@@
 			)
 		)
-		(property "Value" "74LS74"
+		(property "Value" "74HCT74"
 			(at 18.034 146.05 0)
 			(effects
@@
 			)
 		)
-		(property "Value" "74LS08"
+		(property "Value" "74HCT08"
 			(at 73.914 146.05 0)
 			(effects
@@
 			)
 		)
-		(property "Value" "74LS74"
+		(property "Value" "74HCT74"
 			(at 132.334 146.05 0)
 			(effects
@@
 			)
 		)
-		(property "Value" "74F14"
+		(property "Value" "74HCT14"
 			(at 108.458 146.05 0)
 			(effects
@@
 			)
 		)
-		(property "Value" "74LS74"
+		(property "Value" "74HCT74"
 			(at 120.904 146.05 0)
 			(effects
@@
 			)
 		)
-		(property "Value" "74LS32"
+		(property "Value" "74HCT32"
 			(at 51.562 146.304 0)
 			(effects
