File: schematics/EVA1_v2/TRAM.kicad_sch (KiCad schematic)
At the start: 13 parts, among them U1 HY6264AxP, U10 74LS165, U2 74LS573, U3 27C32, U5 74LS245, U6 74LS157, U7 74LS157, U8 74LS157, U9 27C64

Commit message: schematics updated
Connections:
- net +5V: no longer U2.1 (OE)
- net GND: now also U2.1 (OE)
Other:
- note added: "alternate Font ROM"
- note removed: "alternatie Font ROM"
- note removed: "ch: U2 Pin1 to GND!"
Changed lines of the file:
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@@
 		(title "EVA1 (Epson Video Adapter) - Text RAM")
 		(date "2025-01-09")
-		(rev "v0.1")
+		(rev "v0.3")
 		(company "100% Offner")
 		(comment 1 "v0.1: Initial Release")
+		(comment 2 "v0.2: Production version")
+		(comment 3 "v0.3: Redesign with SRAM")
 	)
 	(junction
@@
 	(wire
 		(pts
-			(xy 138.43 128.27) (xy 121.92 128.27)
+			(xy 138.43 128.27) (xy 137.16 128.27)
 		)
 		(stroke
@@
 	(wire
 		(pts
+			(xy 137.16 128.27) (xy 137.16 130.81)
+		)
+		(stroke
+			(width 0)
+			(type default)
+		)
+	)
+	(wire
+		(pts
 			(xy 166.37 125.73) (xy 166.37 120.65)
 		)
@@
 	(wire
 		(pts
-			(xy 121.92 121.92) (xy 121.92 128.27)
-		)
-		(stroke
-			(width 0)
-			(type default)
-		)
-	)
-	(wire
-		(pts
 			(xy 27.94 30.48) (xy 34.29 30.48)
 		)
@@
 		)
 	)
-	(text "ch:\nU2 Pin1 to GND!"
-		(exclude_from_sim no)
-		(at 272.542 173.736 0)
-		(effects
-			(font
-				(size 1.27 1.27)
-			)
-		)
-	)
 	(text "Font\nROM"
 		(exclude_from_sim no)
@@
 		)
 	)
-	(text "alternatie Font ROM"
+	(text "alternate Font ROM"
 		(exclude_from_sim no)
 		(at 138.176 193.802 0)
@@
 	)
 	(symbol
-		(lib_id "power:+5V")
-		(at 121.92 121.92 0)
+		(lib_id "power:GND")
+		(at 52.07 59.69 0)
 		(unit 1)
 		(exclude_from_sim no)
@@
 		(on_board yes)
 		(dnp no)
-		(property "Reference" "#PWR070"
-			(at 121.92 125.73 0)
+		(fields_autoplaced yes)
+		(property "Reference" "#PWR028"
+			(at 52.07 66.04 0)
 			(effects
 				(font
@@
 			)
 		)
-		(property "Value" "+5V"
-			(at 121.92 118.745 0)
+		(property "Value" "GND"
+			(at 52.07 63.8231 0)
 			(effects
 				(font
@@
 		)
 		(property "Footprint" ""
-			(at 121.92 121.92 0)
+			(at 52.07 59.69 0)
 			(effects
 				(font
@@
 		)
 		(property "Datasheet" ""
-			(at 121.92 121.92 0)
+			(at 52.07 59.69 0)
 			(effects
 				(font
@@
 		)
 		(property "Description" ""
-			(at 121.92 121.92 0)
+			(at 52.07 59.69 0)
 			(effects
 				(font
@@
 		)
 		(instances
-			(project "EVA1_production"
+			(project "EVA1"
 				(path "/5be3a086-9309-43f4-b37c-0519e88c3e26/a1f5fccf-e4cd-4d36-afd9-e34a93cb1a3c"
-					(reference "#PWR070")
+					(reference "#PWR028")
 					(unit 1)
 				)
@@
 	(symbol
 		(lib_id "power:GND")
-		(at 52.07 59.69 0)
+		(at 137.16 130.81 0)
 		(unit 1)
 		(exclude_from_sim no)
@@
 		(on_board yes)
 		(dnp no)
-		(fields_autoplaced yes)
-		(property "Reference" "#PWR028"
-			(at 52.07 66.04 0)
+		(property "Reference" "#PWR170"
+			(at 137.16 137.16 0)
 			(effects
 				(font
@@
 		)
 		(property "Value" "GND"
-			(at 52.07 63.8231 0)
+			(at 137.16 134.62 0)
 			(effects
 				(font
@@
 		)
 		(property "Footprint" ""
-			(at 52.07 59.69 0)
+			(at 137.16 130.81 0)
 			(effects
 				(font
@@
 		)
 		(property "Datasheet" ""
-			(at 52.07 59.69 0)
+			(at 137.16 130.81 0)
 			(effects
 				(font
@@
 		)
 		(property "Description" ""
-			(at 52.07 59.69 0)
+			(at 137.16 130.81 0)
 			(effects
 				(font
@@
 		)
 		(instances
-			(project "EVA1"
+			(project "EVA1_v2"
 				(path "/5be3a086-9309-43f4-b37c-0519e88c3e26/a1f5fccf-e4cd-4d36-afd9-e34a93cb1a3c"
-					(reference "#PWR028")
+					(reference "#PWR170")
 					(unit 1)
 				)

Commit message: New version for production
Changed lines of the file:
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@@
 (kicad_sch
-	(version 20231120)
+	(version 20250114)
 	(generator "eeschema")
-	(generator_version "8.0")
+	(generator_version "9.0")
 	(paper "A4")
 	(title_block
@@
 		(comment 3 "v0.3: Redesign with SRAM")
 	)
+	(text "0x1000-0x17FF in Standard EVA1\n0x1000-0x1FFF here."
+		(exclude_from_sim no)
+		(at 162.306 72.898 0)
+		(effects
+			(font
+				(size 1.27 1.27)
+			)
+		)
+	)
+	(text "Font\nROM"
+		(exclude_from_sim no)
+		(at 210.82 113.284 0)
+		(effects
+			(font
+				(size 1.27 1.27)
+			)
+		)
+	)
+	(text "Text\nRAM"
+		(exclude_from_sim no)
+		(at 166.624 43.18 0)
+		(effects
+			(font
+				(size 1.27 1.27)
+			)
+		)
+	)
+	(text "alternate Font ROM"
+		(exclude_from_sim no)
+		(at 138.176 193.802 0)
+		(effects
+			(font
+				(size 1.27 1.27)
+			)
+		)
+	)
 	(junction
 		(at 110.49 182.88)
@@
 		)
 	)
-	(text "0x1000-0x17FF in Standard EVA1\n0x1000-0x1FFF here."
-		(exclude_from_sim no)
-		(at 162.306 72.898 0)
-		(effects
-			(font
-				(size 1.27 1.27)
-			)
-		)
-	)
-	(text "Font\nROM"
-		(exclude_from_sim no)
-		(at 210.82 113.284 0)
-		(effects
-			(font
-				(size 1.27 1.27)
-			)
-		)
-	)
-	(text "Text\nRAM"
-		(exclude_from_sim no)
-		(at 166.624 43.18 0)
-		(effects
-			(font
-				(size 1.27 1.27)
-			)
-		)
-	)
-	(text "alternate Font ROM"
-		(exclude_from_sim no)
-		(at 138.176 193.802 0)
-		(effects
-			(font
-				(size 1.27 1.27)
-			)
-		)
-	)

Commit message: Schematic and Board updated
Parts:
- U10: value 74LS165 -> 74HCT165
- U5: value 74LS245 -> 74HCT245
- U6, U7, U8: value 74LS157 -> 74ALS157
Changed lines of the file:
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@@
 			)
 		)
-		(property "Value" "74LS245"
+		(property "Value" "74HCT245"
 			(at 223.1741 20.32 0)
 			(effects
@@
 			)
 		)
-		(property "Value" "74LS165"
+		(property "Value" "74HCT165"
 			(at 265.0841 85.09 0)
 			(effects
@@
 			)
 		)
-		(property "Value" "74LS157"
+		(property "Value" "74ALS157"
 			(at 63.1541 77.47 0)
 			(effects
@@
 			)
 		)
-		(property "Value" "74LS157"
+		(property "Value" "74ALS157"
 			(at 66.9641 22.86 0)
 			(effects
@@
 			)
 		)
-		(property "Value" "74LS157"
+		(property "Value" "74ALS157"
 			(at 69.5041 128.27 0)
 			(effects
