File: schematics/EVA1_v2/videosignal.kicad_sch (KiCad schematic)
At the start: 20 parts, among them J2 BAS, Q2 BC337, Q3 BC337, U12 74LS32, U18 74LS08, U19 74LS86, U22 74F14, U4 74LS74

Commit message: New version for production
Parts:
- added J11: Conn_Coaxial, my_own_conn:Keystone_RCA-Jack, symbol Connector:Conn_Coaxial
Connections:
- net GND: now also J11.2 (Ext)
- net at J2.1 (Pin_1), Q2.3 (E), R8.1: now also J11.1 (In)
Changed lines of the file:
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@@
 (kicad_sch
-	(version 20231120)
+	(version 20250114)
 	(generator "eeschema")
-	(generator_version "8.0")
+	(generator_version "9.0")
 	(paper "A4")
 	(title_block
@@
 		(comment 3 "v0.3: Redesign with SRAM")
 	)
+	(text "C14 tested with 'LS04 and 4.7nF"
+		(exclude_from_sim no)
+		(at 45.212 47.244 0)
+		(effects
+			(font
+				(size 1.27 1.27)
+			)
+		)
+	)
+	(text "sets Intensity High\nfor Characters with Bit 7 set."
+		(exclude_from_sim no)
+		(at 143.51 148.844 0)
+		(effects
+			(font
+				(size 1.27 1.27)
+			)
+			(justify left)
+		)
+	)
+	(text "sets characters inverse \nwith Bit 7 set"
+		(exclude_from_sim no)
+		(at 143.002 125.476 0)
+		(effects
+			(font
+				(size 1.27 1.27)
+			)
+			(justify left)
+		)
+	)
 	(junction
 		(at 167.64 114.3)
@@
 		(color 0 0 0 0)
 	)
+	(junction
+		(at 254 130.81)
+		(diameter 0)
+		(color 0 0 0 0)
+	)
 	(no_connect
 		(at 144.78 121.92)
@@
 	(wire
 		(pts
+			(xy 254 116.84) (xy 254 130.81)
+		)
+		(stroke
+			(width 0)
+			(type default)
+		)
+	)
+	(wire
+		(pts
 			(xy 124.46 116.84) (xy 127 116.84)
 		)
@@
 	(wire
 		(pts
-			(xy 242.57 130.81) (xy 255.27 130.81)
+			(xy 242.57 130.81) (xy 254 130.81)
 		)
 		(stroke
@@
 	(wire
 		(pts
+			(xy 254 130.81) (xy 255.27 130.81)
+		)
+		(stroke
+			(width 0)
+			(type default)
+		)
+	)
+	(wire
+		(pts
 			(xy 99.06 93.98) (xy 101.6 93.98)
 		)
@@
 	(wire
 		(pts
+			(xy 261.62 116.84) (xy 254 116.84)
+		)
+		(stroke
+			(width 0)
+			(type default)
+		)
+	)
+	(wire
+		(pts
 			(xy 133.35 109.22) (xy 137.16 109.22)
 		)
@@
 		)
 	)
-	(text "C14 tested with 'LS04 and 4.7nF"
-		(exclude_from_sim no)
-		(at 45.212 47.244 0)
-		(effects
-			(font
-				(size 1.27 1.27)
-			)
-		)
-	)
-	(text "sets Intensity High\nfor Characters with Bit 7 set."
-		(exclude_from_sim no)
-		(at 143.51 148.844 0)
-		(effects
-			(font
-				(size 1.27 1.27)
-			)
-			(justify left)
-		)
-	)
-	(text "sets characters inverse \nwith Bit 7 set"
-		(exclude_from_sim no)
-		(at 143.002 125.476 0)
-		(effects
-			(font
-				(size 1.27 1.27)
-			)
-			(justify left)
-		)
-	)
 	(hierarchical_label "~{INV_CHAR}"
 		(shape input)
@@
 					(unit 1)
 				)
+			)
+		)
+	)
+	(symbol
+		(lib_id "Connector:Conn_Coaxial")
+		(at 266.7 116.84 0)
+		(unit 1)
+		(exclude_from_sim no)
+		(in_bom yes)
+		(on_board yes)
+		(dnp no)
+		(fields_autoplaced yes)
+		(property "Reference" "J11"
+			(at 270.51 115.8631 0)
+			(effects
+				(font
+					(size 1.27 1.27)
+				)
+				(justify left)
+			)
+		)
+		(property "Value" "Conn_Coaxial"
+			(at 270.51 118.4031 0)
+			(effects
+				(font
+					(size 1.27 1.27)
+				)
+				(justify left)
+			)
+		)
+		(property "Footprint" "my_own_conn:Keystone_RCA-Jack"
+			(at 266.7 116.84 0)
+			(effects
+				(font
+					(size 1.27 1.27)
+				)
+				(hide yes)
+			)
+		)
+		(property "Datasheet" "~"
+			(at 266.7 116.84 0)
+			(effects
+				(font
+					(size 1.27 1.27)
+				)
+				(hide yes)
+			)
+		)
+		(property "Description" "coaxial connector (BNC, SMA, SMB, SMC, Cinch/RCA, LEMO, ...)"
+			(at 266.7 116.84 0)
+			(effects
+				(font
+					(size 1.27 1.27)
+				)
+				(hide yes)
+			)
+		)
+		(pin "1"
+		)
+		(pin "2"
+		)
+		(instances
+			(project ""
+				(path "/5be3a086-9309-43f4-b37c-0519e88c3e26/71008dda-dbef-4238-9894-aa4b7094e856"
+					(reference "J11")
+					(unit 1)
+				)
+			)
+		)
+	)
+	(symbol
+		(lib_id "power:GND")
+		(at 266.7 121.92 0)
+		(unit 1)
+		(exclude_from_sim no)
+		(in_bom yes)
+		(on_board yes)
+		(dnp no)
+		(fields_autoplaced yes)
+		(property "Reference" "#PWR0134"
+			(at 266.7 128.27 0)
+			(effects
+				(font
+					(size 1.27 1.27)
+				)
+				(hide yes)
+			)
+		)
+		(property "Value" "GND"
+			(at 266.7 126.0531 0)
+			(effects
+				(font
+					(size 1.27 1.27)
+				)
+			)
+		)
+		(property "Footprint" ""
+			(at 266.7 121.92 0)
+			(effects
+				(font
+					(size 1.27 1.27)
+				)
+				(hide yes)
+			)
+		)
+		(property "Datasheet" ""
+			(at 266.7 121.92 0)
+			(effects
+				(font
+					(size 1.27 1.27)
+				)
+				(hide yes)
+			)
+		)
+		(property "Description" ""
+			(at 266.7 121.92 0)
+			(effects
+				(font
+					(size 1.27 1.27)
+				)
+				(hide yes)
+			)
+		)
+		(pin "1"
+		)
+		(instances
+			(project "EVA1_v2"
+				(path "/5be3a086-9309-43f4-b37c-0519e88c3e26/71008dda-dbef-4238-9894-aa4b7094e856"
+					(reference "#PWR0134")
+					(unit 1)
+				)

Commit message: Schematic and Board updated
Parts:
- U12: value 74LS32 -> 74HCT32
- U18: value 74LS08 -> 74HCT08
- U19: value 74LS86 -> 74HCT86
- U22: value 74F14 -> 74HCT14
- U4: value 74LS74 -> 74HCT74
Changed lines of the file:
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@@
 			)
 		)
-		(property "Value" "74F14"
+		(property "Value" "74HCT14"
 			(at 25.4 53.34 0)
 			(effects
@@
 			)
 		)
-		(property "Value" "74LS08"
+		(property "Value" "74HCT08"
 			(at 134.6117 83.82 0)
 			(effects
@@
 			)
 		)
-		(property "Value" "74LS08"
+		(property "Value" "74HCT08"
 			(at 54.6017 73.66 0)
 			(effects
@@
 			)
 		)
-		(property "Value" "74F14"
+		(property "Value" "74HCT14"
 			(at 55.88 53.34 0)
 			(effects
@@
 			)
 		)
-		(property "Value" "74LS08"
+		(property "Value" "74HCT08"
 			(at 81.026 73.152 0)
 			(effects
@@
 			)
 		)
-		(property "Value" "74LS32"
+		(property "Value" "74HCT32"
 			(at 105.41 114.3 0)
 			(effects
@@
 			)
 		)
-		(property "Value" "74LS74"
+		(property "Value" "74HCT74"
 			(at 139.3541 135.89 0)
 			(effects
@@
 			)
 		)
-		(property "Value" "74LS32"
+		(property "Value" "74HCT32"
 			(at 115.824 88.138 0)
 			(effects
@@
 			)
 		)
-		(property "Value" "74LS32"
+		(property "Value" "74HCT32"
 			(at 105.664 137.16 0)
 			(effects
@@
 			)
 		)
-		(property "Value" "74LS08"
+		(property "Value" "74HCT08"
 			(at 93.9717 83.82 0)
 			(effects
@@
 			)
 		)
-		(property "Value" "74LS74"
+		(property "Value" "74HCT74"
 			(at 139.3541 113.03 0)
 			(effects
@@
 			)
 		)
-		(property "Value" "74LS86"
+		(property "Value" "74HCT86"
 			(at 154.6352 109.22 0)
 			(effects
@@
 			)
 		)
-		(property "Value" "74LS86"
+		(property "Value" "74HCT86"
 			(at 45.4152 86.36 0)
 			(effects

Commit message: new Gerber files
Parts:
- renumbered C20 to C114
Changed lines of the file:
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@@
 		(title "EVA1 (Epson Video Adapter) - Video Output")
 		(date "2025-01-09")
-		(rev "v0.3")
+		(rev "v0.5")
 		(company "100% Offner")
-		(comment 1 "v0.1: Initial Release")
-		(comment 2 "v0.2: Production version")
-		(comment 3 "v0.3: Redesign with SRAM")
+		(comment 1 "v0.2: Production version")
+		(comment 2 "v0.3: Redesign with SRAM")
+		(comment 3 "v0.4: Mounting Holes and Buttons position ch.")
+		(comment 4 "v0.5: ch. XTAL to 18M and fixed IC Var. (HCT, F,...), Pulldown on RPi and conn. for Color")
 	)
 	(text "C14 tested with 'LS04 and 4.7nF"
@@
 		(dnp no)
 		(fields_autoplaced yes)
-		(property "Reference" "C20"
+		(property "Reference" "C114"
 			(at 39.37 62.2235 0)
 			(effects
@@
 			(project "EVA1_v2"
 				(path "/5be3a086-9309-43f4-b37c-0519e88c3e26/71008dda-dbef-4238-9894-aa4b7094e856"
-					(reference "C20")
+					(reference "C114")
 					(unit 1)
 				)
